Commit message: turret

File: mark_I/assets/rex_rover.urdf (robot description, URDF)
Before this commit: robot rex_full, 32 links, 31 joints
Links:
- removed link arm_fixed_tip
- removed link arm_moving_tip
- removed link arm_section_5
- added link arm_section_4_ext, mass 0.2; collision cylinder length=0.05 radius=0.02; visual mesh filename=meshes/section_2.obj
- added link turret_drill; visual mesh filename=stl/arm_turret_drill.stl scale=0.002 0.002 0.002
- added link turret_pixl; visual mesh filename=stl/arm_turret_pixl.stl scale=0.0015 0.0015 0.0015
- added link turret_plate; visual mesh filename=stl/arm_turret_gdrt_fcs.stl scale=0.003 0.003 0.003
- added link turret_shwa; visual mesh filename=stl/arm_turret_sherloc_watson.stl scale=0.002 0.002 0.002
- link arm_section_4: geometry collision cylinder length=0.05 radius=0.02; visual mesh filename=meshes/section_1.obj
Joints:
- removed joint arm_t7f
- removed joint arm_t7m
- added joint turret_drill_base: type fixed, parent turret_plate, child turret_drill, origin xyz=0 -0.02 -0.05 rpy=-1.57 0 0, axis 0 0 1
- added joint turret_pixl_base: type fixed, parent turret_drill, child turret_pixl, origin xyz=-0.03 0.075 0.02 rpy=0 0 1.57, axis 0 0 1
- added joint turret_plate_base: type fixed, parent arm_section_4_ext, child turret_plate, origin xyz=0 -0.02 -0.015 rpy=-3.14 0 0, axis 0 0 1, limit lower=-1.57 upper=1.57 effort=100.0 velocity=0.5
- added joint turret_shwa_base: type fixed, parent turret_drill, child turret_shwa, origin xyz=0 0.03 0 rpy=0 0 0, axis 0 0 1
- joint motor_arm_m5: axis 0 0 1 -> 1 0 0; origin xyz=0 -0.048 0 rpy=0 -1.5707963267949 0 -> xyz=0 -0.048 0 rpy=-1.57 0 3.14
- joint motor_arm_m6: axis 0 0 -1 -> 1 0 0; child arm_section_5 -> arm_section_4_ext; limit lower=-0.436 upper=1.5 effort=100.0 velocity=0.7 -> lower=-1.57 upper=1.57 effort=100.0 velocity=0.5; origin xyz=0 -0.058 0 rpy=0 -1.5707963267949 0 -> xyz=0 0 0.05 rpy=0 0 0

Commit message: mastcam

File: mark_I/assets/rex_rover.urdf (robot description, URDF)
Before this commit: robot rex_full, 34 links, 33 joints
Links:
- added link hga_antenna_link; visual mesh filename=stl/hga_antenna.stl scale=0.001 0.001 0.001
- added link hga_base_link; visual mesh filename=stl/hga_base.stl scale=0.001 0.001 0.001
- added link hga_pin_link; visual mesh filename=stl/hga_azimuth_pin.stl scale=0.001 0.001 0.001
- added link mastercam2_rear_link; visual mesh filename=stl/mastcam_z.stl scale=0.0009 0.0009 0.0009
- added link mastercam_front1_link; visual mesh filename=stl/mastcam_z.stl scale=0.00085 0.00085 0.00085
- added link mastercam_rear_link; visual mesh filename=stl/mastcam_z.stl scale=0.0009 0.0009 0.0009
Joints:
- added joint antenna_pin: type fixed, parent hga_pin_link, child hga_antenna_link, origin xyz=0.0019 -0.001 0.021 rpy=0 0 0, axis 0 1 0, limit lower=-3.14 upper=3.14 effort=100.0 velocity=0.7
- added joint hga_base_base: type fixed, parent chassis_front_link, child hga_base_link, origin xyz=0.1303 0.0266 0.043 rpy=0 0 0
- added joint mastercam2_rear_base: type fixed, parent chassis_front_link, child mastercam2_rear_link, origin xyz=0.078 0.018 0.02 rpy=3.14 0.1 0
- added joint mastercam_front1_base: type fixed, parent chassis_front_link, child mastercam_front1_link, origin xyz=-0.09 0 -0.03 rpy=0 0 0
- added joint mastercam_rear_base: type fixed, parent chassis_front_link, child mastercam_rear_link, origin xyz=0.078 -0.02 0.02 rpy=3.14 0.1 0
- added joint pin_base: type fixed, parent hga_base_link, child hga_pin_link, origin xyz=0 -0.0015 -0.01 rpy=0 0 0, axis 0 0 1, limit lower=-3.14 upper=3.14 effort=100.0 velocity=0.7
